Commit message: Fix arm mount orientation: rpy=(0,0,pi/2) so joint1 axis=Z-up, arm extends Y+

File: dk1_dual_arm.urdf (robot description, URDF)
Before this commit: robot dk1_dual_arm, 24 links, 23 joints
Joints:
- joint left_arm_mount: origin xyz=-0.290 0.0 0.040 rpy=1.5707963267948966 0 3.141592653589793 -> xyz=-0.290 0.0 0.040 rpy=0 0 1.5707963267948966
- joint right_arm_mount: origin xyz=0.290 0.0 0.040 rpy=1.5707963267948966 0 3.141592653589793 -> xyz=0.290 0.0 0.040 rpy=0 0 1.5707963267948966

Commit message: Replace mesh geometry with inline boxes for crossbar and camera mast
- front_crossbar: 700x80x40mm box, correct Y/Z position (front face at Y=0, base at Z=0)
- camera_mast: 30x30x400mm box, sits on crossbar top (Z=40mm), center at Z=240mm
- Remove stale .glb/.stl mesh files (no longer referenced)
- Both noted as simplified boxes (real HFS profile has T-slots)

File: dk1_dual_arm.urdf (robot description, URDF)
Before this commit: robot dk1_dual_arm, 26 links, 25 joints
Links:
- link camera_mast: geometry collision box size=0.030 0.030 0.400; visual box size=0.030 0.030 0.400
- link front_crossbar: geometry collision box size=0.700 0.080 0.040; visual box size=0.700 0.080 0.040
Joints:
- joint camera_mast_joint: origin xyz=0 -0.011 0.0 rpy=0 0 0 -> xyz=0.0 0.011 0.240 rpy=0 0 0
- joint front_crossbar_joint: origin xyz=0 0 0.020 rpy=0 0 0 -> xyz=0.0 -0.040 0.020 rpy=0 0 0

Commit message: Fix crossbar Y position: center at Y=0 (aligned with arm mounts)

File: dk1_dual_arm.urdf (robot description, URDF)
Before this commit: robot dk1_dual_arm, 26 links, 25 joints
Joints:
- joint front_crossbar_joint: origin xyz=0.0 -0.040 0.020 rpy=0 0 0 -> xyz=0.0 0.0 0.020 rpy=0 0 0
