Commit message: Add mounting structure geometry: front crossbar and camera mast
Generate parametric box meshes (STL + GLB) for the HFS8-4080-700
front crossbar and HFS6-3030-400 camera mast, and add them as
fixed links in the URDF.

Co-Authored-By: Claude Opus 4.6 <noreply@anthropic.com>

File: dk1_dual_arm.urdf (robot description, URDF)
Before this commit: robot dk1_dual_arm, 24 links, 23 joints
Links:
- added link camera_mast; collision mesh filename=meshes/camera_mast.stl; visual mesh filename=meshes/camera_mast.glb
- added link front_crossbar; collision mesh filename=meshes/front_crossbar.stl; visual mesh filename=meshes/front_crossbar.glb
Joints:
- added joint camera_mast_joint: type fixed, parent world, child camera_mast, origin xyz=0 -0.011 0.0 rpy=0 0 0
- added joint front_crossbar_joint: type fixed, parent world, child front_crossbar, origin xyz=0 0 0.020 rpy=0 0 0

Commit message: Clean up repo: move meshes to top-level, remove helper scripts and submodule
Move arm meshes from trlc-dk1 submodule into meshes/{visual,collision}/,
update URDF paths, and remove unnecessary files (create_mounting_meshes.py,
validate_urdf.py, step_analysis.md, trlc-dk1 submodule).

Co-Authored-By: Claude Opus 4.6 (1M context) <noreply@anthropic.com>

File: dk1_dual_arm.urdf (robot description, URDF)
Before this commit: robot dk1_dual_arm, 26 links, 25 joints
Links:
- link left_base_link: geometry collision mesh filename=meshes/collision/base_link.stl; visual mesh filename=meshes/visual/base_link.glb
- link left_finger_left: geometry collision mesh filename=meshes/collision/finger_left.stl; visual mesh filename=meshes/visual/finger_left.glb
- link left_finger_right: geometry collision mesh filename=meshes/collision/finger_right.stl; visual mesh filename=meshes/visual/finger_right.glb
- link left_link1-2: geometry collision mesh filename=meshes/collision/link1-2.stl; visual mesh filename=meshes/visual/link1-2.glb
- link left_link2-3: geometry collision mesh filename=meshes/collision/link2-3.stl; visual mesh filename=meshes/visual/link2-3.glb
- link left_link3-4: geometry collision mesh filename=meshes/collision/link3-4.stl; visual mesh filename=meshes/visual/link3-4.glb
- link left_link4-5: geometry collision mesh filename=meshes/collision/link4-5.stl; visual mesh filename=meshes/visual/link4-5.glb
- link left_link5-6: geometry collision mesh filename=meshes/collision/link5-6.stl; visual mesh filename=meshes/visual/link5-6.glb
- link left_link6-7: geometry collision mesh filename=meshes/collision/link6-7.stl; visual mesh filename=meshes/visual/link6-7.glb
- link right_base_link: geometry collision mesh filename=meshes/collision/base_link.stl; visual mesh filename=meshes/visual/base_link.glb
- link right_finger_left: geometry collision mesh filename=meshes/collision/finger_left.stl; visual mesh filename=meshes/visual/finger_left.glb
- link right_finger_right: geometry collision mesh filename=meshes/collision/finger_right.stl; visual mesh filename=meshes/visual/finger_right.glb
- link right_link1-2: geometry collision mesh filename=meshes/collision/link1-2.stl; visual mesh filename=meshes/visual/link1-2.glb
- link right_link2-3: geometry collision mesh filename=meshes/collision/link2-3.stl; visual mesh filename=meshes/visual/link2-3.glb
- link right_link3-4: geometry collision mesh filename=meshes/collision/link3-4.stl; visual mesh filename=meshes/visual/link3-4.glb
- link right_link4-5: geometry collision mesh filename=meshes/collision/link4-5.stl; visual mesh filename=meshes/visual/link4-5.glb
- link right_link5-6: geometry collision mesh filename=meshes/collision/link5-6.stl; visual mesh filename=meshes/visual/link5-6.glb
- link right_link6-7: geometry collision mesh filename=meshes/collision/link6-7.stl; visual mesh filename=meshes/visual/link6-7.glb

Commit message: Rename tool0 links to tcp; add flange tool0 frames (both arms)
For both right_ and left_ arms, the link named tool0 actually sat at the
+0.158m fingertip grasp point — semantically the TCP, not the ROS-Industrial
flange frame. Rename those to {side}_tcp / {side}_tcp_joint and add separate
{side}_tool0 frames at the link6-7 (flange) origin so cartesian actions can
use a zero-lever effector frame decoupled from wrist-rotation lever.

Co-Authored-By: Claude Opus 4.8 (1M context) <noreply@anthropic.com>

File: dk1_dual_arm.urdf (robot description, URDF)
Before this commit: robot dk1_dual_arm, 26 links, 25 joints
Links:
- added link left_tcp
- added link right_tcp
Joints:
- removed joint left_gripper_tool0
- removed joint right_gripper_tool0
- added joint left_tcp_joint: type fixed, parent left_link6-7, child left_tcp, origin xyz=0.158 0 0 rpy=-1.5707963267948966 0 -1.5707963267948966
- added joint left_tool0_joint: type fixed, parent left_link6-7, child left_tool0, origin xyz=0 0 0 rpy=-1.5707963267948966 0 -1.5707963267948966
- added joint right_tcp_joint: type fixed, parent right_link6-7, child right_tcp, origin xyz=0.158 0 0 rpy=-1.5707963267948966 0 -1.5707963267948966
- added joint right_tool0_joint: type fixed, parent right_link6-7, child right_tool0, origin xyz=0 0 0 rpy=-1.5707963267948966 0 -1.5707963267948966

Commit message: Move tcp to grasp point 5mm before finger tips; add fingertips_center (both arms)
tcp and fingertips_center are now children of tool0, so their offsets are pure
translations along tool-z and the orientation convention is defined once per arm.
tcp moves to 0.153 (5mm before the tips); fingertips_center keeps the tip plane
at 0.158.

Co-Authored-By: Claude Opus 4.8 (1M context) <noreply@anthropic.com>

File: dk1_dual_arm.urdf (robot description, URDF)
Before this commit: robot dk1_dual_arm, 28 links, 27 joints
Links:
- added link left_fingertips_center
- added link right_fingertips_center
Joints:
- added joint left_fingertips_center_joint: type fixed, parent left_tool0, child left_fingertips_center, origin xyz=0 0 0.158 rpy=0 0 0
- added joint right_fingertips_center_joint: type fixed, parent right_tool0, child right_fingertips_center, origin xyz=0 0 0.158 rpy=0 0 0
- joint left_tcp_joint: origin xyz=0.158 0 0 rpy=-1.5707963267948966 0 -1.5707963267948966 -> xyz=0 0 0.153 rpy=0 0 0; parent left_link6-7 -> left_tool0
- joint right_tcp_joint: origin xyz=0.158 0 0 rpy=-1.5707963267948966 0 -1.5707963267948966 -> xyz=0 0 0.153 rpy=0 0 0; parent right_link6-7 -> right_tool0

Commit message: Remove fingertips_center frames; note tip plane in tcp comments
Only 5mm from tcp — consumers compute offsets along tool-z from tcp anyway,
and two near-identical effector frames invite ambiguity about the canonical
action frame. The tip plane (0.158) is documented in the tcp comments.

Co-Authored-By: Claude Opus 4.8 (1M context) <noreply@anthropic.com>

File: dk1_dual_arm.urdf (robot description, URDF)
Before this commit: robot dk1_dual_arm, 30 links, 29 joints
Links:
- removed link left_fingertips_center
- removed link right_fingertips_center
Joints:
- removed joint left_fingertips_center_joint
- removed joint right_fingertips_center_joint

Commit message: Update camera link poses to calibrated estimates
overhead_camera, left_camera, right_camera joint origins replaced with the poses
our calibration produced (flywheel extrinsics.json): head_cam_in_base for the
overhead cam, cam_in_link6-7 = tool0_in_link6-7 @ cam2ee for the wrists. Each link
frame is the calibrated OpenCV optical frame — for the upside-down wrist cams that
is the 180°-rotated (upright/teleop) frame cam2ee is calibrated in. The old nominal
CAD values (wrist ones were in a mechanical frame, wrongly oriented) are kept in
XML comments.

Co-Authored-By: Claude Opus 4.8 <noreply@anthropic.com>

File: dk1_dual_arm.urdf (robot description, URDF)
Before this commit: robot dk1_dual_arm, 28 links, 27 joints
Joints:
- joint left_camera_joint: origin xyz=0.0471 0 0.063314 rpy=0 0.2618 0 -> xyz=0.049037 -0.002560 0.051802 rpy=-1.749208 0.018688 -1.552414
- joint overhead_camera_mount: origin xyz=0.0 0.01065 0.47881 rpy=-2.356194490192345 0 0 -> xyz=-0.005139 0.015259 0.469202 rpy=-2.303446 -0.002141 -0.017958
- joint right_camera_joint: origin xyz=0.0471 0 0.063314 rpy=0 0.2618 0 -> xyz=0.043612 0.000394 0.049776 rpy=-1.749933 -0.028894 -1.569908

Commit message: Update left wrist camera pose to FR-008 auto-calibration
left_camera_joint origin refreshed from the 50-pose active wrist auto-calibration (reproj 0.194px). Right wrist unchanged.

Co-Authored-By: Claude Opus 4.8 <noreply@anthropic.com>

File: dk1_dual_arm.urdf (robot description, URDF)
Before this commit: robot dk1_dual_arm, 28 links, 27 joints
Joints:
- joint left_camera_joint: origin xyz=0.049037 -0.002560 0.051802 rpy=-1.749208 0.018688 -1.552414 -> xyz=0.050555 0.000134 0.052583 rpy=-1.733395 0.028466 -1.555563

Commit message: Update right wrist camera pose to FR-008 auto-calibration
right_camera_joint origin from the 50-pose right-wrist hand-eye (41/50, PARK 0.220px, spread 5.13mm). Mirrors the vendored copy in flywheel. Right only; left unchanged.

Co-Authored-By: Claude Opus 4.8 <noreply@anthropic.com>

File: dk1_dual_arm.urdf (robot description, URDF)
Before this commit: robot dk1_dual_arm, 28 links, 27 joints
Joints:
- joint right_camera_joint: origin xyz=0.043612 0.000394 0.049776 rpy=-1.749933 -0.028894 -1.569908 -> xyz=0.046026 -0.000806 0.047603 rpy=-1.746946 -0.021432 -1.563364

Commit message: Update right wrist camera pose (FR-008 hand-eye on refit intrinsics)
right_camera_joint from the right hand-eye re-run on the refit intrinsics (PARK 0.162px, spread 4.22mm). Mirrors the vendored copy in flywheel.

Co-Authored-By: Claude Opus 4.8 <noreply@anthropic.com>

File: dk1_dual_arm.urdf (robot description, URDF)
Before this commit: robot dk1_dual_arm, 28 links, 27 joints
Joints:
- joint right_camera_joint: origin xyz=0.046026 -0.000806 0.047603 rpy=-1.746946 -0.021432 -1.563364 -> xyz=0.048136 0.000649 0.050856 rpy=-1.734517 -0.011914 -1.579281

Commit message: Update left wrist camera pose (FR-008 hand-eye on refit intrinsics)
left_camera_joint from the left hand-eye re-run on the refit intrinsics (PARK 0.191px); adopted for cross-arm consistency with the right (fx~458, pose 2.5mm/2.1deg). Mirrors the vendored copy.

Co-Authored-By: Claude Opus 4.8 <noreply@anthropic.com>

File: dk1_dual_arm.urdf (robot description, URDF)
Before this commit: robot dk1_dual_arm, 28 links, 27 joints
Joints:
- joint left_camera_joint: origin xyz=0.050555 0.000134 0.052583 rpy=-1.733395 0.028466 -1.555563 -> xyz=0.050209 -0.000553 0.050161 rpy=-1.715683 0.013687 -1.560020
